File: footprint_family/MSOP/osh-park_2_layer_standard_order.kicad_pcb (KiCad board)
At the start: 2 copper layers, 0 parts

Commit message: Schematic and layout for MSOP chips.
Parts:
- added P1: CONN_01X05, pins:pin-1x05-sq, F.Cu at (139.7, 106.7)
- added P2: CONN_01X05, pins:pin-1x05, F.Cu at (154.9, 106.7)
- added R1: R, Resistors_SMD:R_0805_HandSoldering, B.Cu at (147.3, 106.7)
- added R2: R, Resistors_SMD:R_0805_HandSoldering, B.Cu at (147.3, 109.2)
- added R3: R, Resistors_SMD:R_0805_HandSoldering, B.Cu at (147.3, 111.8)
- added R4: R, Resistors_SMD:R_0805_HandSoldering, B.Cu at (147.3, 114.3)
- added R5: R, Resistors_SMD:R_0805_HandSoldering, B.Cu at (147.3, 116.8)
- added U1: IC10, footprints:MSOP-10, F.Cu at (147.3, 111.8)
Routing:
- net Net-(P1-Pad5): track 0.00 -> 13.3 mm
- net Net-(P1-Pad1): track 0.00 -> 13.3 mm
- net Net-(P2-Pad5): track 0.00 -> 13.3 mm
- net Net-(P2-Pad1): track 0.00 -> 13.3 mm
- net Net-(P1-Pad4): track 0.00 -> 12.5 mm
- net Net-(P1-Pad2): track 0.00 -> 12.5 mm
- net Net-(P2-Pad4): track 0.00 -> 12.5 mm
- net Net-(P2-Pad2): track 0.00 -> 12.5 mm
- net Net-(P1-Pad3): track 0.00 -> 11.7 mm
- net Net-(P2-Pad3): track 0.00 -> 11.7 mm
Other:
- board outline added: 19.1 x 14 mm

Commit message: Smaller PCB for MSOP
Parts:
- moved P1 1.27 mm to (141.0, 106.7)
- moved P2 1.27 mm to (153.7, 106.7)
Routing:
- net Net-(P2-Pad4): track 12.5 -> 9.94 mm
- net Net-(P2-Pad3): track 11.7 -> 9.15 mm
- net Net-(P2-Pad2): track 12.5 -> 9.94 mm
- net Net-(P1-Pad5): track 13.3 -> 10.7 mm
- net Net-(P1-Pad4): track 12.5 -> 9.94 mm
- net Net-(P1-Pad3): track 11.7 -> 9.15 mm
- net Net-(P1-Pad2): track 12.5 -> 9.94 mm
- net Net-(P1-Pad1): track 13.3 -> 10.7 mm
- net Net-(P2-Pad1): track 13.3 -> 10.7 mm
- net Net-(P2-Pad5): track 13.3 -> 10.7 mm
Other:
- board size 19.1 x 14 mm -> 16.5 x 14 mm
Changed lines of the file:
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@@
     (36 B.SilkS user)
     (37 F.SilkS user)
-    (38 B.Mask user hide)
-    (39 F.Mask user hide)
+    (38 B.Mask user)
+    (39 F.Mask user)
     (40 Dwgs.User user)
     (41 Cmts.User user)
@@
   )
   (module pins:pin-1x05-sq (layer F.Cu)
-    (at 139.7 106.68)
+    (at 140.97 106.68)
     (descr "Header pin. 2.54mm pitch. 1mm drills. Shape 1x05. Square pin 1.")
     (tags "pin header")
@@
   )
   (module pins:pin-1x05 (layer F.Cu)
-    (at 154.94 106.68)
+    (at 153.67 106.68)
     (descr "Header pin. 2.54mm pitch. 1mm drills. Shape 1x05.")
     (tags "pin header")
@@
       (net 4 "Net-(P1-Pad4)"))
   )
-  (gr_line (start 156.845 104.775) (end 137.795 104.775) (angle 90) (layer Edge.Cuts) (width 0.127))
-  (gr_line (start 156.845 118.745) (end 156.845 104.775) (angle 90) (layer Edge.Cuts) (width 0.127))
-  (gr_line (start 137.795 118.745) (end 156.845 118.745) (angle 90) (layer Edge.Cuts) (width 0.127))
-  (gr_line (start 137.795 104.775) (end 137.795 118.745) (angle 90) (layer Edge.Cuts) (width 0.127))
-  (segment (start 139.7 106.68) (end 145.97 106.68) (width 1) (layer B.Cu) (net 1))
-  (segment (start 145.12 110.49) (end 143.51 110.49) (width 0.25) (layer F.Cu) (net 1))
-  (segment (start 143.51 110.49) (end 139.7 106.68) (width 0.25) (layer F.Cu) (net 1))
-  (segment (start 145.97 109.22) (end 139.7 109.22) (width 1) (layer B.Cu) (net 2))
-  (segment (start 145.12 111.125) (end 141.605 111.125) (width 0.25) (layer F.Cu) (net 2))
-  (segment (start 141.605 111.125) (end 139.7 109.22) (width 0.25) (layer F.Cu) (net 2))
-  (segment (start 139.7 111.76) (end 145.97 111.76) (width 1) (layer B.Cu) (net 3))
-  (segment (start 145.12 111.76) (end 139.7 111.76) (width 0.25) (layer F.Cu) (net 3))
-  (segment (start 145.97 114.3) (end 139.7 114.3) (width 1) (layer B.Cu) (net 4))
-  (segment (start 145.12 112.395) (end 141.605 112.395) (width 0.25) (layer F.Cu) (net 4))
-  (segment (start 141.605 112.395) (end 139.7 114.3) (width 0.25) (layer F.Cu) (net 4))
-  (segment (start 139.7 116.84) (end 145.97 116.84) (width 1) (layer B.Cu) (net 5))
-  (segment (start 145.12 113.03) (end 143.51 113.03) (width 0.25) (layer F.Cu) (net 5))
-  (segment (start 143.51 113.03) (end 139.7 116.84) (width 0.25) (layer F.Cu) (net 5))
-  (segment (start 148.67 106.68) (end 154.94 106.68) (width 1) (layer B.Cu) (net 6))
-  (segment (start 149.52 110.49) (end 151.13 110.49) (width 0.25) (layer F.Cu) (net 6))
-  (segment (start 151.13 110.49) (end 154.94 106.68) (width 0.25) (layer F.Cu) (net 6))
-  (segment (start 154.94 109.22) (end 148.67 109.22) (width 1) (layer B.Cu) (net 7))
-  (segment (start 149.52 111.125) (end 153.035 111.125) (width 0.25) (layer F.Cu) (net 7))
-  (segment (start 153.035 111.125) (end 154.94 109.22) (width 0.25) (layer F.Cu) (net 7))
-  (segment (start 148.67 111.76) (end 154.94 111.76) (width 1) (layer B.Cu) (net 8))
-  (segment (start 149.52 111.76) (end 154.94 111.76) (width 0.25) (layer F.Cu) (net 8))
-  (segment (start 154.94 114.3) (end 148.67 114.3) (width 1) (layer B.Cu) (net 9))
-  (segment (start 149.52 112.395) (end 153.035 112.395) (width 0.25) (layer F.Cu) (net 9))
-  (segment (start 153.035 112.395) (end 154.94 114.3) (width 0.25) (layer F.Cu) (net 9))
-  (segment (start 148.67 116.84) (end 154.94 116.84) (width 1) (layer B.Cu) (net 10))
-  (segment (start 149.52 113.03) (end 151.13 113.03) (width 0.25) (layer F.Cu) (net 10))
-  (segment (start 151.13 113.03) (end 154.94 116.84) (width 0.25) (layer F.Cu) (net 10))
+  (gr_line (start 139.065 118.745) (end 139.065 104.775) (angle 90) (layer Edge.Cuts) (width 0.127))
+  (gr_line (start 155.575 118.745) (end 139.065 118.745) (angle 90) (layer Edge.Cuts) (width 0.127))
+  (gr_line (start 155.575 104.775) (end 155.575 118.745) (angle 90) (layer Edge.Cuts) (width 0.127))
+  (gr_line (start 139.065 104.775) (end 155.575 104.775) (angle 90) (layer Edge.Cuts) (width 0.127))
+  (segment (start 140.97 106.68) (end 145.97 106.68) (width 1) (layer B.Cu) (net 1) (status C00000))
+  (segment (start 145.12 110.49) (end 144.78 110.49) (width 0.25) (layer F.Cu) (net 1) (status C00000))
+  (segment (start 144.78 110.49) (end 140.97 106.68) (width 0.25) (layer F.Cu) (net 1) (status C00000))
+  (segment (start 145.97 109.22) (end 140.97 109.22) (width 1) (layer B.Cu) (net 2) (status C00000))
+  (segment (start 145.12 111.125) (end 142.875 111.125) (width 0.25) (layer F.Cu) (net 2) (status 400000))
+  (segment (start 142.875 111.125) (end 140.97 109.22) (width 0.25) (layer F.Cu) (net 2) (status 800000))
+  (segment (start 140.97 111.76) (end 145.97 111.76) (width 1) (layer B.Cu) (net 3) (status C00000))
+  (segment (start 145.12 111.76) (end 140.97 111.76) (width 0.25) (layer F.Cu) (net 3) (status C00000))
+  (segment (start 145.97 114.3) (end 140.97 114.3) (width 1) (layer B.Cu) (net 4) (status C00000))
+  (segment (start 145.12 112.395) (end 142.875 112.395) (width 0.25) (layer F.Cu) (net 4) (status 400000))
+  (segment (start 142.875 112.395) (end 140.97 114.3) (width 0.25) (layer F.Cu) (net 4) (status 800000))
+  (segment (start 140.97 116.84) (end 145.97 116.84) (width 1) (layer B.Cu) (net 5) (status C00000))
+  (segment (start 145.12 113.03) (end 144.78 113.03) (width 0.25) (layer F.Cu) (net 5) (status C00000))
+  (segment (start 144.78 113.03) (end 140.97 116.84) (width 0.25) (layer F.Cu) (net 5) (status C00000))
+  (segment (start 148.67 106.68) (end 153.67 106.68) (width 1) (layer B.Cu) (net 6) (status C00000))
+  (segment (start 149.52 110.49) (end 149.86 110.49) (width 0.25) (layer F.Cu) (net 6) (status C00000))
+  (segment (start 149.86 110.49) (end 153.67 106.68) (width 0.25) (layer F.Cu) (net 6) (status C00000))
+  (segment (start 153.67 109.22) (end 148.67 109.22) (width 1) (layer B.Cu) (net 7) (status C00000))
+  (segment (start 149.52 111.125) (end 151.765 111.125) (width 0.25) (layer F.Cu) (net 7) (status 400000))
+  (segment (start 151.765 111.125) (end 153.67 109.22) (width 0.25) (layer F.Cu) (net 7) (status 800000))
+  (segment (start 148.67 111.76) (end 153.67 111.76) (width 1) (layer B.Cu) (net 8) (status C00000))
+  (segment (start 149.52 111.76) (end 153.67 111.76) (width 0.25) (layer F.Cu) (net 8) (status C00000))
+  (segment (start 153.67 114.3) (end 148.67 114.3) (width 1) (layer B.Cu) (net 9) (status C00000))
+  (segment (start 149.52 112.395) (end 151.765 112.395) (width 0.25) (layer F.Cu) (net 9) (status 400000))
+  (segment (start 151.765 112.395) (end 153.67 114.3) (width 0.25) (layer F.Cu) (net 9) (status 800000))
+  (segment (start 148.67 116.84) (end 153.67 116.84) (width 1) (layer B.Cu) (net 10) (status C00000))
+  (segment (start 149.52 113.03) (end 149.86 113.03) (width 0.25) (layer F.Cu) (net 10) (status C00000))
+  (segment (start 149.86 113.03) (end 153.67 116.84) (width 0.25) (layer F.Cu) (net 10) (status C00000))
 )
